Commit message: adjusted mismatched package names

File: src/r-gator-simulator-2/r-gator-model-2/urdf/rgator_model.urdf.xacro (robot description, xacro)
@@ -1,5 +1,5 @@
 <?xml version="1.0" ?>
 <!-- =================================================================================== -->
-<!-- |    This document was autogenerated by xacro from rgator_model.urdf              | -->
+<!-- |    This document was autogenerated by xacro from r-gator-model-2.urdf              | -->
 <!-- |    EDITING THIS FILE BY HAND IS NOT RECOMMENDED                                 | -->
 <!-- =================================================================================== -->
@@ -7,7 +7,7 @@
      Commit Version: 1.6.0-4-g7f85cfe  Build Version: 1.6.7995.38578
      For more information, please see http://wiki.ros.org/sw_urdf_exporter -->
-<robot name="rgator_model" xmlns:xacro="http://www.ros.org/wiki/xacro">
-    <xacro:include filename="$(find rgator_model)/urdf/rgator.gazebo" />
-    <xacro:include filename="$(find rgator_model)/urdf/macros.xacro" />
+<robot name="r-gator-model-2" xmlns:xacro="http://www.ros.org/wiki/xacro">
+    <xacro:include filename="$(find r-gator-model-2)/urdf/rgator.gazebo" />
+    <xacro:include filename="$(find r-gator-model-2)/urdf/macros.xacro" />
     <xacro:arg name="velodyne_points" default="false"/>
     <xacro:arg name="laser_points" default="false"/>
@@ -33,5 +33,5 @@
         <origin rpy="0 0 0" xyz="0 0 0"/>
         <geometry>
-            <mesh filename="package://rgator_model/meshes/base_link.STL"/>
+            <mesh filename="package://r-gator-model-2/meshes/base_link.STL"/>
         </geometry>
         <material name="">
@@ -42,5 +42,5 @@
         <origin rpy="0 0 0" xyz="0 0 0"/>
         <geometry>
-            <mesh filename="package://rgator_model/meshes/base_link.STL"/>
+            <mesh filename="package://r-gator-model-2/meshes/base_link.STL"/>
         </geometry>
         </collision>
@@ -77,14 +77,14 @@
         <origin rpy="0 0 0" xyz="0 0 0"/>
         <geometry>
-            <mesh filename="package://rgator_model/meshes/front_left_wheel_link.STL"/>
-        </geometry>
-        <material name="">
-            <color rgba="0.250980392156863 0.250980392156863 0.250980392156863 1"/>
-        </material>
-        </visual>
-        <collision>
-        <origin rpy="0 0 0" xyz="0 0 0"/>
-        <geometry>
-            <mesh filename="package://rgator_model/meshes/front_left_wheel_link.STL"/>
+            <mesh filename="package://r-gator-model-2/meshes/front_left_wheel_link.STL"/>
+        </geometry>
+        <material name="">
+            <color rgba="0.250980392156863 0.250980392156863 0.250980392156863 1"/>
+        </material>
+        </visual>
+        <collision>
+        <origin rpy="0 0 0" xyz="0 0 0"/>
+        <geometry>
+            <mesh filename="package://r-gator-model-2/meshes/front_left_wheel_link.STL"/>
         </geometry>
         </collision>
@@ -122,14 +122,14 @@
         <origin rpy="0 0 0" xyz="0 0 0"/>
         <geometry>
-            <mesh filename="package://rgator_model/meshes/front_right_wheel_link.STL"/>
-        </geometry>
-        <material name="">
-            <color rgba="0.250980392156863 0.250980392156863 0.250980392156863 1"/>
-        </material>
-        </visual>
-        <collision>
-        <origin rpy="0 0 0" xyz="0 0 0"/>
-        <geometry>
-            <mesh filename="package://rgator_model/meshes/front_right_wheel_link.STL"/>
+            <mesh filename="package://r-gator-model-2/meshes/front_right_wheel_link.STL"/>
+        </geometry>
+        <material name="">
+            <color rgba="0.250980392156863 0.250980392156863 0.250980392156863 1"/>
+        </material>
+        </visual>
+        <collision>
+        <origin rpy="0 0 0" xyz="0 0 0"/>
+        <geometry>
+            <mesh filename="package://r-gator-model-2/meshes/front_right_wheel_link.STL"/>
         </geometry>
         </collision>
@@ -153,14 +153,14 @@
         <origin rpy="0 0 0" xyz="0 0 0"/>
         <geometry>
-            <mesh filename="package://rgator_model/meshes/middle_left_wheel_link.STL"/>
-        </geometry>
-        <material name="">
-            <color rgba="0.250980392156863 0.250980392156863 0.250980392156863 1"/>
-        </material>
-        </visual>
-        <collision>
-        <origin rpy="0 0 0" xyz="0 0 0"/>
-        <geometry>
-            <mesh filename="package://rgator_model/meshes/middle_left_wheel_link.STL"/>
+            <mesh filename="package://r-gator-model-2/meshes/middle_left_wheel_link.STL"/>
+        </geometry>
+        <material name="">
+            <color rgba="0.250980392156863 0.250980392156863 0.250980392156863 1"/>
+        </material>
+        </visual>
+        <collision>
+        <origin rpy="0 0 0" xyz="0 0 0"/>
+        <geometry>
+            <mesh filename="package://r-gator-model-2/meshes/middle_left_wheel_link.STL"/>
         </geometry>
         </collision>
@@ -184,14 +184,14 @@
         <origin rpy="0 0 0" xyz="0 0 0"/>
         <geometry>
-            <mesh filename="package://rgator_model/meshes/middle_right_wheel_link.STL"/>
-        </geometry>
-        <material name="">
-            <color rgba="0.250980392156863 0.250980392156863 0.250980392156863 1"/>
-        </material>
-        </visual>
-        <collision>
-        <origin rpy="0 0 0" xyz="0 0 0"/>
-        <geometry>
-            <mesh filename="package://rgator_model/meshes/middle_right_wheel_link.STL"/>
+            <mesh filename="package://r-gator-model-2/meshes/middle_right_wheel_link.STL"/>
+        </geometry>
+        <material name="">
+            <color rgba="0.250980392156863 0.250980392156863 0.250980392156863 1"/>
+        </material>
+        </visual>
+        <collision>
+        <origin rpy="0 0 0" xyz="0 0 0"/>
+        <geometry>
+            <mesh filename="package://r-gator-model-2/meshes/middle_right_wheel_link.STL"/>
         </geometry>
         </collision>
@@ -215,14 +215,14 @@
         <origin rpy="0 0 0" xyz="0 0 0"/>
         <geometry>
-            <mesh filename="package://rgator_model/meshes/rear_left_wheel_link.STL"/>
-        </geometry>
-        <material name="">
-            <color rgba="0.250980392156863 0.250980392156863 0.250980392156863 1"/>
-        </material>
-        </visual>
-        <collision>
-        <origin rpy="0 0 0" xyz="0 0 0"/>
-        <geometry>
-            <mesh filename="package://rgator_model/meshes/rear_left_wheel_link.STL"/>
+            <mesh filename="package://r-gator-model-2/meshes/rear_left_wheel_link.STL"/>
+        </geometry>
+        <material name="">
+            <color rgba="0.250980392156863 0.250980392156863 0.250980392156863 1"/>
+        </material>
+        </visual>
+        <collision>
+        <origin rpy="0 0 0" xyz="0 0 0"/>
+        <geometry>
+            <mesh filename="package://r-gator-model-2/meshes/rear_left_wheel_link.STL"/>
         </geometry>
         </collision>
@@ -246,14 +246,14 @@
         <origin rpy="0 0 0" xyz="0 0 0"/>
         <geometry>
-            <mesh filename="package://rgator_model/meshes/rear_right_wheel_link.STL"/>
-        </geometry>
-        <material name="">
-            <color rgba="0.250980392156863 0.250980392156863 0.250980392156863 1"/>
-        </material>
-        </visual>
-        <collision>
-        <origin rpy="0 0 0" xyz="0 0 0"/>
-        <geometry>
-            <mesh filename="package://rgator_model/meshes/rear_right_wheel_link.STL"/>
+            <mesh filename="package://r-gator-model-2/meshes/rear_right_wheel_link.STL"/>
+        </geometry>
+        <material name="">
+            <color rgba="0.250980392156863 0.250980392156863 0.250980392156863 1"/>
+        </material>
+        </visual>
+        <collision>
+        <origin rpy="0 0 0" xyz="0 0 0"/>
+        <geometry>
+            <mesh filename="package://r-gator-model-2/meshes/rear_right_wheel_link.STL"/>
         </geometry>
         </collision>
