Commit message: Update r_gator_velodyne.rviz, fix some urdf problems

File: src/r-gator-simulator-2/r-gator-model-2/urdf/rgator_model.urdf (robot description, URDF)
Before this commit: robot rgator_model, 10 links, 9 joints
Links:
- added link world
- link base_link: geometry collision mesh filename=package://r-gator-model-2/meshes/base_link.STL; visual mesh filename=package://r-gator-model-2/meshes/base_link.STL
- link front_left_wheel_link: geometry collision mesh filename=package://r-gator-model-2/meshes/front_left_wheel_link.STL; visual mesh filename=package://r-gator-model-2/meshes/front_left_wheel_link.STL
- link front_right_wheel_link: geometry collision mesh filename=package://r-gator-model-2/meshes/front_right_wheel_link.STL; visual mesh filename=package://r-gator-model-2/meshes/front_right_wheel_link.STL
- link middle_left_wheel_link: geometry collision mesh filename=package://r-gator-model-2/meshes/middle_left_wheel_link.STL; visual mesh filename=package://r-gator-model-2/meshes/middle_left_wheel_link.STL
- link middle_right_wheel_link: geometry collision mesh filename=package://r-gator-model-2/meshes/middle_right_wheel_link.STL; visual mesh filename=package://r-gator-model-2/meshes/middle_right_wheel_link.STL
- link rear_left_wheel_link: geometry collision mesh filename=package://r-gator-model-2/meshes/rear_left_wheel_link.STL; visual mesh filename=package://r-gator-model-2/meshes/rear_left_wheel_link.STL
- link rear_right_wheel_link: geometry collision mesh filename=package://r-gator-model-2/meshes/rear_right_wheel_link.STL; visual mesh filename=package://r-gator-model-2/meshes/rear_right_wheel_link.STL
Joints:
- added joint world_link: type fixed, parent world, child base_link, origin xyz=0 0 0 rpy=0 0 0

Commit message: fixed r-gator clipping issue

File: src/r-gator-simulator-2/r-gator-model-2/urdf/rgator_model.urdf (robot description, URDF)
Before this commit: robot rgator_model, 11 links, 10 joints
Links:
- removed link GPS_link
- removed link IMU_link
- removed link world
Joints:
- removed joint GPS_joint
- removed joint IMU_joint
- removed joint world_link
